File: schematics/gateway/gateway.kicad_sch (KiCad schematic)
At the start: 12 parts, among them J1 Power, J2 PN532_Port, J4 Button_Port

Commit message: adjust pad sizes for easier drilling and soldering
Parts:
- J1: footprint TerminalBlock:TerminalBlock_Xinya_XY308-2.54-2P_1x02_P2.54mm_Horizontal -> TerminalBlock:TerminalBlock_MaiXu_MX126-5.0-02P_1x02_P5.00mm
Changed lines of the file:
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@@
 			)
 		)
-		(property "Footprint" "TerminalBlock:TerminalBlock_Xinya_XY308-2.54-2P_1x02_P2.54mm_Horizontal"
+		(property "Footprint" "TerminalBlock:TerminalBlock_MaiXu_MX126-5.0-02P_1x02_P5.00mm"
 			(at 24.13 25.146 0)
 			(hide yes)
