File: schematics/telemetry/telemetry.kicad_pcb (KiCad board)
At the start: 2 copper layers, 81 x 90 mm, 19 parts, among them J1 Power, J2 PN532_Port, J3 LED_Port, J4 Button_Port, J5 PZEM_Port, J6 Relay_Port, K1 Relay, Q1 IRLZ44N, U1 ESP32S3, U2 LoRa

Commit message: adjust pad sizes for easier drilling and soldering
Parts:
- J1: footprint TerminalBlock:TerminalBlock_Xinya_XY308-2.54-2P_1x02_P2.54mm_Horizontal -> TerminalBlock:TerminalBlock_MaiXu_MX126-5.0-02P_1x02_P5.00mm
- moved J3 1.50 mm to (89.5, 45.5)
- moved J4 1.50 mm to (89.5, 37.5)
Routing:
- net GND: track 249.5 -> 245.3 mm
- net Net-(J3-Pin_3): track 12.2 -> 14.0 mm
- net Net-(J4-Pin_1): track 16.9 -> 18.6 mm
- net Net-(J3-Pin_1): track 10.8 -> 12.3 mm
Other:
- board text added: "+"
- board text added: "-"
